File: Combined_PowerSupply_v0.1/Combined_PowerSupply_v0.1.kicad_sch (KiCad schematic)
At the start: 62 parts, among them CN1 C3697-WJ2EDGRC-5.08-02P-14-00A, CN10 C71370-WJ2EDGK-5.08-02P-14-00A, CN11 C3697-WJ2EDGRC-5.08-02P-14-00A, CN12 C71370-WJ2EDGK-5.08-02P-14-00A, CN2 C71370-WJ2EDGK-5.08-02P-14-00A, CN3 C3697-WJ2EDGRC-5.08-02P-14-00A, CN4 C71370-WJ2EDGK-5.08-02P-14-00A, CN5 C3697-WJ2EDGRC-5.08-02P-14-00A, CN6 C71370-WJ2EDGK-5.08-02P-14-00A, CN7 C3697-WJ2EDGRC-5.08-02P-14-00A, CN8 C71370-WJ2EDGK-5.08-02P-14-00A, CN9 C3697-WJ2EDGRC-5.08-02P-14-00A, J1 C698356-09031646921, U1 C507146-LM7805S_TR, U2 C40133-MP4560DN-LF-Z, U3 C507195-LM7815S_TR, U4 C5145368-LM7812SRG, U5 C259972-LM1084S-3.3_TR, U6 C492421-PZ254V-12-8P, U7 C492421-PZ254V-12-8P

Commit message: Commit fixes
Parts:
- removed G1: IAMSnanofiber, IAMS:IAMSnanofiber, symbol IAMS:IAMSnanofiber
- removed G2: IAMS, IAMS:IAMS, symbol IAMS:IAMS
- removed G3: IAMSYb, IAMS:IAMSYb, symbol IAMS:IAMSYb
